Commit message: 修改：固定一端近轨

File: src/wr_description/urdf/wr_chassis.urdf.xacro (robot description, xacro)
@@ -154,5 +154,5 @@
   <joint name="mid360_joint" type="fixed">
     <parent link="base_link"/><child link="mid360_link"/>
-    <origin xyz="0 0 0.46" rpy="0 0 0"/>
+    <origin xyz="0 0 0.46" rpy="0 0.785398163 0"/>
   </joint>
   <link name="front_camera_link"/>

Commit message: feat: 建立轮轨人物跟随导航基础框架

File: src/wr_description/urdf/wr_chassis.urdf.xacro (robot description, xacro)
@@ -161,8 +161,3 @@
     <origin xyz="0.39 0 0.31" rpy="0 0 0"/>
   </joint>
-  <link name="rear_camera_link"/>
-  <joint name="rear_camera_joint" type="fixed">
-    <parent link="base_link"/><child link="rear_camera_link"/>
-    <origin xyz="-0.39 0 0.31" rpy="0 0 3.141592654"/>
-  </joint>
 </robot>

Commit message: 重新确定技术路线

File: src/wr_description/urdf/wr_chassis.urdf.xacro (robot description, xacro)
@@ -32,5 +32,5 @@
       <material name="chassis_grey"/>
     </visual>
-    <!-- Convex primitives are used for stable simulation; the detailed STL remains visual-only. -->
+    <!-- 凸基本几何体用于稳定物理仿真；高精度 STL 仅用于外观显示。 -->
     <collision>
       <origin xyz="0 0 0.17" rpy="0 0 0"/>
@@ -143,5 +143,5 @@
     wheel_ixx="0.00461473" wheel_ixy="0.00000094" wheel_ixz="0.00001332"
     wheel_iyy="0.00458059" wheel_iyz="0.00000388" wheel_izz="0.00710833"/>
-  <!-- Provisional sensor frames. Measure and replace these xyz/rpy values on the real chassis. -->
+  <!-- 传感器坐标系暂定值；实车安装后必须测量并替换 xyz/rpy。 -->
   <link name="imu_link"/>
   <joint name="imu_joint" type="fixed">
@@ -154,5 +154,5 @@
   <joint name="mid360_joint" type="fixed">
     <parent link="base_link"/><child link="mid360_link"/>
-    <origin xyz="0 0 0.46" rpy="0 0.785398163 0"/>
+    <origin xyz="0 0 0.46" rpy="0 0.349065850 0"/>
   </joint>
   <link name="front_camera_link"/>

File: src/wr_description/urdf/wr_chassis_mock_control.urdf.xacro (robot description, xacro)
@@ -15,6 +15,6 @@
       <joint name="${prefix}_steering_joint">
         <command_interface name="position">
-          <param name="min">-1.745329252</param>
-          <param name="max">1.745329252</param>
+          <param name="min">-2.88</param>
+          <param name="max">2.88</param>
         </command_interface>
         <state_interface name="position"><param name="initial_value">0.0</param></state_interface>
